Commit message: Added backwing with aerodynamics; added fidelity visuals

File: mrg_modimoop_description/urdf/mrg_modimoop.urdf.xacro (robot description, xacro)
@@ -10,4 +10,5 @@
   <!-- ===================== -->
   <xacro:property name="mesh_scale" value="0.001 0.001 0.001"/>
+  <xacro:property name="backwing_mesh_scale" value="0.0004 0.0004 0.0004"/>
   <!-- Rough masses (kg). Replace with measured values -->
   <xacro:property name="m_hull"     value="20.0"/>
@@ -15,4 +16,9 @@
   <xacro:property name="m_wingsail" value="1.0"/>
   <xacro:property name="m_rudder"   value="0.1"/>
+  <xacro:property name="m_backwing" value="0.2"/>
+  <xacro:property name="rudder_rod_radius" value="0.0045"/>
+  <xacro:property name="wingsail_rod_radius" value="0.01"/>
+  <xacro:property name="backwing_rod_radius" value="0.008"/>
+  <xacro:property name="rod_mass" value="0.001"/>
   <!-- Simple diagonal inertias (kg·m²). Replace with real inertias -->
   <xacro:property name="I_small" value="0.02"/>
@@ -22,4 +28,5 @@
   <material name="Red"><color rgba="0.8 0.2 0.2 1.0"/></material>
   <material name="Black"><color rgba="0.05 0.05 0.05 1.0"/></material>
+  <material name="Pink"><color rgba="1.0 0.2 0.6 1.0"/></material>
   <!-- ===================== -->
   <!-- Links                 -->
@@ -37,5 +44,5 @@
         <mesh filename="package://mrg_modimoop_description/models/mrg_modimoop_base/hull/hull.STL" scale="${mesh_scale}"/>
       </geometry>
-      <material name="Grey"/>
+      <material name="Pink"/>
     </visual>
     <collision name="hull_collision">
@@ -49,17 +56,17 @@
   <link name="wingsail">
     <inertial>
-      <origin xyz="0.125 0.034 0.5" rpy="0 0 0"/>
+      <origin xyz="0.15 0.034 0.5" rpy="0 0 0"/>
       <mass value="${m_wingsail}"/>
       <inertia ixx="${I_small}" ixy="0.0" ixz="0.0" iyy="${I_small}" iyz="0.0" izz="${I_small}"/>
     </inertial>
     <visual>
-      <origin xyz="-0.05 -0.015 0" rpy="0 0 0"/>
+      <origin xyz="-0.025 -0.015 0" rpy="0 0 0"/>
       <geometry>
         <mesh filename="package://mrg_modimoop_description/models/mrg_modimoop_base/mainsail/mainsail.STL" scale="${mesh_scale}"/>
       </geometry>
-      <material name="Red"/>
+      <material name="Pink"/>
     </visual>
     <collision name="wingsail_collision">
-      <origin xyz="0.12 0.03 0.675" rpy="0 0 0"/>
+      <origin xyz="0.15 0.03 0.675" rpy="0 0 0"/>
       <geometry>
         <!-- chord, thickness, height (meters) -->
@@ -68,4 +75,26 @@
     </collision>
   </link>
+  <link name="backwing">
+    <inertial>
+      <!-- <origin xyz="0.25 0.02 0.2" rpy="0 0 0"/> -->
+      <origin xyz="0 0 0" rpy="0 0 0"/>
+      <mass value="${m_backwing}"/>
+      <inertia ixx="${I_small}" ixy="0.0" ixz="0.0" iyy="${I_small}" iyz="0.0" izz="${I_small}"/>
+    </inertial>
+    <visual>
+      <origin xyz="0 0 0" rpy="0 0 0"/>
+      <geometry>
+        <mesh filename="package://mrg_modimoop_description/models/mrg_modimoop_base/mainsail/mainsail.STL" scale="${backwing_mesh_scale}"/>
+      </geometry>
+      <material name="Pink"/>
+    </visual>
+    <collision name="backwing_collision">
+      <origin xyz="0.07 0.03 0.25" rpy="0 0 0"/>
+      <geometry>
+        <!-- chord, thickness, height (meters) -->
+        <box size="0.13 0.02 0.5"/>
+      </geometry>
+    </collision>
+  </link>
   <!-- Rudder (revolute about vertical axis) -->
   <link name="rudder">
@@ -73,5 +102,5 @@
       <origin xyz="0 0.08 -0.08" rpy="0 0 0"/>
       <mass value="${m_rudder}"/>
-      <inertia ixx="$0.0" ixy="0.0" ixz="0.0" iyy="$0.0" iyz="0.0" izz="$0.0"/>
+      <inertia ixx="0.0" ixy="0.0" ixz="0.0" iyy="0.0" iyz="0.0" izz="0.0"/>
     </inertial>
     <visual>
@@ -105,5 +134,5 @@
         <mesh filename="package://mrg_modimoop_description/models/mrg_modimoop_base/keel/keel_plate.STL" scale="${mesh_scale}"/>
       </geometry>
-      <material name="Blue"/>
+      <material name="Grey"/>
     </visual>
     <!-- Bulb visual -->
@@ -114,5 +143,5 @@
         <mesh filename="package://mrg_modimoop_description/models/mrg_modimoop_base/keel/keel_bulb.STL" scale="${mesh_scale}"/>
       </geometry>
-      <material name="Blue"/>
+      <material name="Grey"/>
     </visual>
     <!-- Plate collision -->
@@ -150,4 +179,18 @@
     <dynamics damping="0.2" friction="0.0"/>
   </joint>
+  <link name="backwing_hinge"/>
+  <joint name="backwing_hinge_joint" type="fixed">
+    <parent link="wingsail"/>
+    <child link="backwing_hinge"/>
+    <origin xyz="0.45 0.0125 0.4" rpy="0 0 0"/>
+  </joint>
+  <joint name="backwing_joint" type="continuous">
+    <parent link="backwing_hinge"/>
+    <child link="backwing"/>
+    <origin xyz="0 0 0" rpy="0 0 0"/>
+    <!-- coaxial -->
+    <axis xyz="0 0 1"/>
+    <dynamics damping="0.05" friction="0.0"/>
+  </joint>
   <!-- Rudder rotates around Z for yaw -->
   <joint name="rudder_joint" type="continuous">
@@ -158,4 +201,81 @@
     <dynamics damping="0.1" friction="0.0"/>
   </joint>
+  <link name = "rudder_rod">
+    <inertial>
+      <origin xyz="0 0 0" rpy = "0 0 0"/>
+      <mass value="${rod_mass}"/>
+      <inertia ixx="1e-6" ixy="0" ixz="0" iyy="1e-6" iyz="0" izz="1e-6"/>
+    </inertial>
+    <visual>
+      <origin xyz="0 0 0" rpy="0 0 0"/>
+      <geometry>
+        <cylinder radius="${rudder_rod_radius}" length="0.20"/>
+      </geometry>
+      <material name="Black"/>
+    </visual>
+  </link>
+  <joint name="rudder_rod_mount" type="fixed">
+    <parent link="hull"/>
+    <child link="rudder_rod"/>
+    <origin xyz="0.175 -0.3 0.3" rpy="0 0 0"/>
+  </joint>
+  <link name="wingsail_rod">
+    <inertial>
+      <origin xyz="0 0 0" rpy="0 0 0"/>
+      <mass value="${rod_mass}"/>
+      <inertia ixx="1e-6" ixy="0" ixz="0" iyy="1e-6" iyz="0" izz="1e-6"/>
+    </inertial>
+    <visual>
+      <origin xyz="0 0.01 0" rpy="0 0 0"/>
+      <geometry>
+        <cylinder radius="${wingsail_rod_radius}" length="0.40"/>
+      </geometry>
+      <material name="Black"/>
+    </visual>
+  </link>
+  <joint name="wingsail_rod_mount" type="fixed">
+    <parent link="hull"/>
+    <child link="wingsail_rod"/>
+    <origin xyz="0.2 -0.65 0.65" rpy="0 0 1.570796"/>
+  </joint>
+  <link name="backwing_rod_top">
+    <inertial>
+      <origin xyz="0 0 0" rpy="0 0 0"/>
+      <mass value="${rod_mass}"/>
+      <inertia ixx="1e-6" ixy="0" ixz="0" iyy="1e-6" iyz="0" izz="1e-6"/>
+    </inertial>
+    <visual>
+      <!-- Rotate cylinder so it runs along X -->
+      <origin xyz="0 0.008 0.7" rpy="0 1.570796 0"/>
+      <geometry>
+        <cylinder radius="${backwing_rod_radius}" length="0.425"/>
+      </geometry>
+      <material name="Black"/>
+    </visual>
+  </link>
+  <link name="backwing_rod_bottom">
+    <inertial>
+      <origin xyz="0 0 0" rpy="0 0 0"/>
+      <mass value="${rod_mass}"/>
+      <inertia ixx="1e-6" ixy="0" ixz="0" iyy="1e-6" iyz="0" izz="1e-6"/>
+    </inertial>
+    <visual>
+      <origin xyz="0 0.008 0.35" rpy="0 1.570796 0"/>
+      <geometry>
+        <cylinder radius="${backwing_rod_radius}" length="0.425"/>
+      </geometry>
+      <material name="Black"/>
+    </visual>
+  </link>
+  <joint name="backwing_rod_top_mount" type="fixed">
+    <parent link="wingsail"/>
+    <child link="backwing_rod_top"/>
+    <origin xyz="0.25 0.02 0.2" rpy="0 0 0"/>
+  </joint>
+  <joint name="backwing_rod_bottom_mount" type="fixed">
+    <parent link="wingsail"/>
+    <child link="backwing_rod_bottom"/>
+    <origin xyz="0.25 0.02 0.05" rpy="0 0 0"/>
+  </joint>
   <!-- ===================== -->
   <!-- Sensor frame links    -->
@@ -189,29 +309,19 @@
   <gazebo reference="wingsail">
     <enable_wind>true</enable_wind>
-    <plugin filename="gz-sim-lift-drag-system" name="gz::sim::systems::LiftDrag">
-      <!-- Fluid / wind -->
-      <air_density>1.225</air_density>          <!-- kg/m^3 -->
-      <wind_velocity>0 0 0</wind_velocity>      <!-- world frame; set nonzero for steady wind -->
-      <!-- Geometry / scaling -->
-      <area>0.35</area>                          <!-- m^2, effective planform area -->
-      <chord>0.25</chord>                        <!-- m, typical sail chord -->
-      <aspect_ratio>3.0</aspect_ratio>           <!-- span^2 / area -->
-      <!-- Orientation: expressed in the wingsail_link frame -->
-      <forward>1 0 0</forward>                   <!-- chord direction -->
-      <upward>0 0 1</upward>                     <!-- span direction -->
-      <!-- Aerodynamic center of pressure (in link frame) -->
-      <cp>0 0 0.4</cp>                           <!-- tweak: typically mid-height and near 1/4 chord -->
-      <!-- Basic coeff model -->
-      <cla>5.5</cla>                             <!-- lift slope (per rad); ~2*pi is 6.28, 5–6 is typical -->
-      <cda>0.8</cda>                             <!-- drag at high AoA, tune -->
-      <cma>0.0</cma>                             <!-- pitching moment slope, optional -->
-      <alpha0>0.0</alpha0>                       <!-- zero-lift AoA (rad) -->
-      <stall_angle>0.45</stall_angle>            <!-- rad (~26 deg) -->
-      <stall_angle2>-0.45</stall_angle2>
-      <cla_stall>1.0</cla_stall>                 <!-- post-stall slope (smaller) -->
-      <cla_stall2>-1.0</cla_stall2>
-      <!-- Optional limits -->
-      <a0>0.0</a0>                                <!-- sometimes used by older variants -->
-      <linkname>wingsail</linkname>
+    <plugin name="gz::sim::systems::SailLiftDrag"
+            filename="asv_sim2-sail-lift-drag-system">
+          <a0>0.0</a0>
+          <cla>6.2832</cla>
+          <alpha_stall>0.1592</alpha_stall>
+          <cla_stall>-0.7083</cla_stall>
+          <cda>0.63662</cda>
+          <area>0.17</area>
+          <fluid_density>1.225</fluid_density>
+          <forward>1 0 0</forward>
+          <upward>0 1 0</upward>
+          <cp>0 0 0</cp>
+          <link_name>wingsail</link_name>
+          <radial_symmetry>1</radial_symmetry>
+          <topic>wingsail/lift_drag</topic>
     </plugin>
     <plugin
@@ -221,4 +331,28 @@
     </plugin>
   </gazebo>
+  <gazebo reference="backwing">
+    <enable_wind>true</enable_wind>
+    <plugin name="gz::sim::systems::SailLiftDrag"
+            filename="asv_sim2-sail-lift-drag-system">
+          <a0>0.0</a0>
+          <cla>6.2832</cla>
+          <alpha_stall>0.1592</alpha_stall>
+          <cla_stall>-0.7083</cla_stall>
+          <cda>0.63662</cda>
+          <area>0.05</area>
+          <fluid_density>1.225</fluid_density>
+          <forward>1 0 0</forward>
+          <upward>0 1 0</upward>
+          <cp>0 0 0</cp>
+          <link_name>backwing</link_name>
+          <radial_symmetry>1</radial_symmetry>
+          <topic>backwing/lift_drag</topic>
+    </plugin>
+    <plugin
+        filename="gz-sim-apply-joint-force-system"
+        name="gz::sim::systems::ApplyJointForce">
+        <joint_name>backwing_joint</joint_name>
+    </plugin>
+  </gazebo>
     <!-- ===================== -->
   <!-- Gazebo sensors        -->
@@ -230,5 +364,5 @@
       <update_rate>200</update_rate>
       <visualize>0</visualize>
-      <!-- Noise models are optional; start clean -->
+      <topic>/modimoop/imu</topic>
       <imu>
         <angular_velocity>
@@ -263,4 +397,5 @@
       <always_on>1</always_on>
       <update_rate>10</update_rate>
+      <topic>/modimoop/navsat</topic>
       <visualize>0</visualize>
     </sensor>
@@ -272,4 +407,5 @@
       <update_rate>50</update_rate>
       <visualize>0</visualize>
+      <topic>/modimoop/mag</topic>
       <magnetometer/>
     </sensor>
@@ -280,4 +416,6 @@
       <joint_name>wingsail_joint</joint_name>
       <joint_name>rudder_joint</joint_name>
+      <joint_name>backwing_joint</joint_name>
+      <topic>/modimoop/joint_state</topic>
       <update_rate>50</update_rate>
     </plugin>

Commit message: Initial commit; branch for testing higher fidelity waves and hydrodynamics

File: mrg_modimoop_description/urdf/mrg_modimoop.urdf.xacro (robot description, xacro)
@@ -12,9 +12,9 @@
   <xacro:property name="backwing_mesh_scale" value="0.0004 0.0004 0.0004"/>
   <!-- Rough masses (kg). Replace with measured values -->
-  <xacro:property name="m_hull"     value="20.0"/>
-  <xacro:property name="m_keel"     value="40.0"/>        <!-- total for keel (plate+bulb) if single link -->
-  <xacro:property name="m_wingsail" value="1.0"/>
-  <xacro:property name="m_rudder"   value="0.1"/>
-  <xacro:property name="m_backwing" value="0.2"/>
+  <xacro:property name="m_hull"     value="22.83"/>
+  <xacro:property name="m_keel"     value="0.01"/>        <!-- total for keel (plate+bulb) if single link -->
+  <xacro:property name="m_wingsail" value="4.44"/>
+  <xacro:property name="m_rudder"   value="0.34"/>
+  <xacro:property name="m_backwing" value="0.17"/>
   <xacro:property name="rudder_rod_radius" value="0.0045"/>
   <xacro:property name="wingsail_rod_radius" value="0.01"/>
@@ -33,9 +33,10 @@
   <!-- ===================== -->
   <!-- Hull is the base -->
+  <!-- Hull is the base -->
   <link name="hull">
     <inertial>
-      <origin xyz="0.175 -0.55 0.45" rpy="1.570796 0 1.570796"/>
+      <origin xyz="0.175 -0.55 0.15" rpy="0 0 0"/>
       <mass value="${m_hull}"/>
-      <inertia ixx="4.848" ixy="0" ixz="0" iyy="7.847" iyz="0" izz="5.3975"/>
+      <inertia ixx="3.70506895" ixy="-0.00022839" ixz="-0.00008461" iyy="0.96696277" iyz="-0.64724529" izz="2.83543540"/>
     </inertial>
     <visual>
@@ -58,5 +59,5 @@
       <origin xyz="0.15 0.034 0.5" rpy="0 0 0"/>
       <mass value="${m_wingsail}"/>
-      <inertia ixx="${I_small}" ixy="0.0" ixz="0.0" iyy="${I_small}" iyz="0.0" izz="${I_small}"/>
+      <inertia ixx="0.78628153" ixy="-0.00004262" ixz="-0.00044123" iyy="0.32623116" iyz="-0.05493911" izz="0.46187925"/>
     </inertial>
     <visual>
@@ -77,8 +78,7 @@
   <link name="backwing">
     <inertial>
-      <!-- <origin xyz="0.25 0.02 0.2" rpy="0 0 0"/> -->
-      <origin xyz="0 0 0" rpy="0 0 0"/>
+      <origin xyz="0.025 0.02 0.2" rpy="0 0 0"/>
       <mass value="${m_backwing}"/>
-      <inertia ixx="${I_small}" ixy="0.0" ixz="0.0" iyy="${I_small}" iyz="0.0" izz="${I_small}"/>
+      <inertia ixx="0.00415255" ixy="0.00000002" ixz="0" iyy="0.00011550" iyz="-0.00000140" izz="0.00405022"/>
     </inertial>
     <visual>
@@ -102,5 +102,5 @@
       <origin xyz="0 0.08 -0.08" rpy="0 0 0"/>
       <mass value="${m_rudder}"/>
-      <inertia ixx="0.0" ixy="0.0" ixz="0.0" iyy="0.0" iyz="0.0" izz="0.0"/>
+      <inertia ixx="0.00323999" ixy="0.00000021" ixz="0.00000004" iyy="0.00089298" iyz="0.00069153" izz="0.00234885"/>
     </inertial>
     <visual>
@@ -123,5 +123,5 @@
     <inertial>
       <!-- Set the CoM where you expect the keel COM; adjust for your CAD -->
-      <origin xyz="0.175 -0.55 0.1" rpy="1.570796 0 0"/>
+      <origin xyz="0.175 -0.55 0.1" rpy="0 0 0"/>
       <mass value="${m_keel}"/>
       <inertia ixx="${m_keel*0.016}" ixy="0.0" ixz="0.0" iyy="${m_keel*0.016}" iyz="0.0" izz="${m_keel*0.016}"/>
@@ -317,7 +317,7 @@
           <area>0.17</area>
           <fluid_density>1.225</fluid_density>
-          <forward>1 0 0</forward>
+          <forward>-1 0 0</forward>
           <upward>0 1 0</upward>
-          <cp>0 0 0</cp>
+          <cp>0.15 0.034 0.5</cp>
           <link_name>wingsail</link_name>
           <radial_symmetry>1</radial_symmetry>
@@ -333,7 +333,7 @@
           <area>0.05</area>
           <fluid_density>1.225</fluid_density>
-          <forward>1 0 0</forward>
+          <forward>-1 0 0</forward>
           <upward>0 1 0</upward>
-          <cp>0 0 0</cp>
+          <cp>0.025 0.02 0.2</cp>
           <link_name>backwing</link_name>
           <radial_symmetry>1</radial_symmetry>
@@ -349,7 +349,7 @@
           <area>0.17</area>
           <fluid_density>1000</fluid_density>
-          <forward>1 0 0</forward>
-          <upward>0 1 0</upward>
-          <cp>0 0 0</cp>
+          <forward>0 -1 0</forward>
+          <upward>1 0 0</upward>
+          <cp>0.175 -0.55 0.1</cp>
           <link_name>keel</link_name>
           <radial_symmetry>1</radial_symmetry>
@@ -365,7 +365,7 @@
           <area>0.12</area>
           <fluid_density>1000</fluid_density>
-          <forward>1 0 0</forward>
-          <upward>0 1 0</upward>
-          <cp>-0.06 0 -0.2</cp>
+          <forward>0 -1 0</forward>
+          <upward>1 0 0</upward>
+          <cp>0 0.08 -0.08</cp>
           <link_name>rudder</link_name>
           <radial_symmetry>1</radial_symmetry>

Commit message: Corrected visuals and inertias

File: mrg_modimoop_description/urdf/mrg_modimoop.urdf.xacro (robot description, xacro)
@@ -57,5 +57,5 @@
   <link name="wingsail">
     <inertial>
-      <origin xyz="0.15 0.034 0.5" rpy="0 0 0"/>
+      <origin xyz="0.15 0.034 0.5" rpy="1.570796 0 1.570796"/>
       <mass value="${m_wingsail}"/>
       <inertia ixx="0.78628153" ixy="-0.00004262" ixz="-0.00044123" iyy="0.32623116" iyz="-0.05493911" izz="0.46187925"/>
@@ -78,12 +78,12 @@
   <link name="backwing">
     <inertial>
-      <origin xyz="0.025 0.02 0.2" rpy="0 0 0"/>
+      <origin xyz="0.025 0.02 0.2" rpy="1.570796 0 1.570796"/>
       <mass value="${m_backwing}"/>
       <inertia ixx="0.00415255" ixy="0.00000002" ixz="0" iyy="0.00011550" iyz="-0.00000140" izz="0.00405022"/>
     </inertial>
     <visual>
-      <origin xyz="0 0 0" rpy="0 0 0"/>
-      <geometry>
-        <mesh filename="package://mrg_modimoop_description/models/mrg_modimoop_base/mainsail/mainsail.STL" scale="${backwing_mesh_scale}"/>
+      <origin xyz="-1.3 0.015 -0.5" rpy="1.570796 0 1.570796"/>
+      <geometry>
+        <mesh filename="package://mrg_modimoop_description/models/mrg_modimoop_base/tailwing/tailwing.STL" scale="${mesh_scale}"/>
       </geometry>
       <material name="Pink"/>
@@ -93,5 +93,5 @@
       <geometry>
         <!-- chord, thickness, height (meters) -->
-        <box size="0.13 0.02 0.5"/>
+        <box size="0.11 0.02 0.55"/>
       </geometry>
     </collision>
@@ -127,19 +127,10 @@
       <inertia ixx="${m_keel*0.016}" ixy="0.0" ixz="0.0" iyy="${m_keel*0.016}" iyz="0.0" izz="${m_keel*0.016}"/>
     </inertial>
-    <!-- Plate visual -->
+    <!-- Keel visual -->
     <visual>
       <!-- Align to plate’s CAD frame relative to keel link frame -->
-      <origin xyz="0.175 -0.7 0.44" rpy="0 1.570796 0"/>
-      <geometry>
-        <mesh filename="package://mrg_modimoop_description/models/mrg_modimoop_base/keel/keel_plate.STL" scale="${mesh_scale}"/>
-      </geometry>
-      <material name="Grey"/>
-    </visual>
-    <!-- Bulb visual -->
-    <visual>
-      <!-- Align bulb mesh relative to keel link frame -->
-      <origin xyz="0.135 -0.21 0.015" rpy="1.570796 0 0"/>
-      <geometry>
-        <mesh filename="package://mrg_modimoop_description/models/mrg_modimoop_base/keel/keel_bulb.STL" scale="${mesh_scale}"/>
+      <origin xyz="0.175 -1.15 0.7" rpy="1.570796 0 3.14159"/>
+      <geometry>
+        <mesh filename="package://mrg_modimoop_description/models/mrg_modimoop_base/keel/keel.STL" scale="${mesh_scale}"/>
       </geometry>
       <material name="Grey"/>
@@ -147,16 +138,16 @@
     <!-- Plate collision -->
     <collision name="keel_plate_collision">
-      <origin xyz="0.175 -0.55 0.34" rpy="0 0 1.570796"/>
+      <origin xyz="0.175 -0.55 0.3" rpy="0 0 1.570796"/>
       <geometry>
         <!-- chord, thickness, span (meters) — tune -->
-        <box size="0.25 0.0125 0.50"/>
+        <box size="0.175 0.0125 0.70"/>
       </geometry>
     </collision>
     <!-- Bulb collision -->
     <collision name="keel_bulb_collision">
-      <origin xyz="0.18 -0.575 0.06" rpy="1.570796 0 0"/>
+      <origin xyz="0.175 -0.565 -0.08" rpy="1.570796 0 0"/>
       <geometry>
         <!-- length is along cylinder Z axis in its collision frame -->
-        <cylinder length="0.7" radius="0.04"/>
+        <cylinder length="0.325" radius="0.045"/>
       </geometry>
     </collision>
@@ -247,7 +238,7 @@
     <visual>
       <!-- Rotate cylinder so it runs along X -->
-      <origin xyz="0 0.008 0.7" rpy="0 1.570796 0"/>
-      <geometry>
-        <cylinder radius="${backwing_rod_radius}" length="0.425"/>
+      <origin xyz="-0.1 0.008 0.73" rpy="0 1.570796 0"/>
+      <geometry>
+        <cylinder radius="${backwing_rod_radius}" length="0.625"/>
       </geometry>
       <material name="Black"/>
@@ -261,7 +252,7 @@
     </inertial>
     <visual>
-      <origin xyz="0 0.008 0.35" rpy="0 1.570796 0"/>
-      <geometry>
-        <cylinder radius="${backwing_rod_radius}" length="0.425"/>
+      <origin xyz="-0.1 0.008 0.32" rpy="0 1.570796 0"/>
+      <geometry>
+        <cylinder radius="${backwing_rod_radius}" length="0.625"/>
       </geometry>
       <material name="Black"/>

Commit message: Added models and custom_waves model for our world; will allow for better performance when actually running sim tests since we don't have to render the visual waves

File: mrg_modimoop_description/urdf/mrg_modimoop.urdf.xacro (robot description, xacro)
@@ -33,8 +33,10 @@
   <!-- ===================== -->
   <!-- Hull is the base -->
-  <!-- Hull is the base -->
   <link name="hull">
     <inertial>
+      <!--<origin xyz="0	0.75915	-1.33874" rpy="0 0 0"/>-->
       <origin xyz="0.175 -0.55 0.15" rpy="0 0 0"/>
+      <!--<origin xyz="0.175 -1.1 0.575" rpy="0 0 0"/>-->
+      <!--<origin xyz="0.175 -0.34085 0.575" rpy="0 0 0"/>-->
       <mass value="${m_hull}"/>
       <inertia ixx="3.70506895" ixy="-0.00022839" ixz="-0.00008461" iyy="0.96696277" iyz="-0.64724529" izz="2.83543540"/>
@@ -122,6 +124,6 @@
   <link name="keel">
     <inertial>
-      <!-- Set the CoM where you expect the keel COM; adjust for your CAD -->
-      <origin xyz="0.175 -0.55 0.1" rpy="0 0 0"/>
+      <!-- Set the CoM where you expect the keel COM; adjust for your CAD --> <!-- 0.175 -0.55 0.1 -->
+      <origin xyz="0 0 0" rpy="0 0 0"/>
       <mass value="${m_keel}"/>
       <inertia ixx="${m_keel*0.016}" ixy="0.0" ixz="0.0" iyy="${m_keel*0.016}" iyz="0.0" izz="${m_keel*0.016}"/>
@@ -130,5 +132,5 @@
     <visual>
       <!-- Align to plate’s CAD frame relative to keel link frame -->
-      <origin xyz="0.175 -1.15 0.7" rpy="1.570796 0 3.14159"/>
+      <origin xyz="0 0 0" rpy="1.570796 0 3.14159"/>
       <geometry>
         <mesh filename="package://mrg_modimoop_description/models/mrg_modimoop_base/keel/keel.STL" scale="${mesh_scale}"/>
@@ -160,5 +162,5 @@
     <parent link="hull"/>
     <child link="keel"/>
-    <origin xyz="0 0 -0.1" rpy="0 0 0"/>
+    <origin xyz="0.175 -1.15 0.7" rpy="0 0 0"/>
   </joint>
   <!-- Wingsail rotates around Z (trim). Limit range ±90° by default -->
