Commit message: Reworked hull, wingsail, backwing, and keel such that all of their local frames are the same; x is the chord direction and x,y,z follow the right-hand rule for all frames.

File: mrg_modimoop_description/urdf/mrg_modimoop.urdf.xacro (robot description, xacro)
@@ -35,6 +35,6 @@
   <link name="hull">
     <inertial>
-      <!--<origin xyz="0	0.75915	-1.33874" rpy="0 0 0"/>-->
-      <origin xyz="0.175 -0.55 0.15" rpy="0 0 0"/>
+      <!--<origin xyz="0 0.75915 -1.33874" rpy="0 0 0"/>-->
+      <origin xyz="0.175 -0.55 0.15" rpy="0 0 1.570796"/>
       <!--<origin xyz="0.175 -1.1 0.575" rpy="0 0 0"/>-->
       <!--<origin xyz="0.175 -0.34085 0.575" rpy="0 0 0"/>-->
@@ -43,5 +43,5 @@
     </inertial>
     <visual>
-      <origin xyz="0 0 0" rpy="1.570796 0 0"/>
+      <origin xyz="-0.41 -0.725 0" rpy="1.570796 0 1.570796"/>
       <geometry>
         <mesh filename="package://mrg_modimoop_description/models/mrg_modimoop_base/hull/hull.STL" scale="${mesh_scale}"/>
@@ -50,5 +50,5 @@
     </visual>
     <collision name="hull_collision">
-      <origin xyz="0.178 -0.55 0.45" rpy="0 0 1.570796"/>
+      <origin xyz="0.178 -0.55 0.45" rpy="0 0 3.14159"/>
       <geometry>
         <box size="1.125 0.35 0.25"/>
@@ -59,10 +59,12 @@
   <link name="wingsail">
     <inertial>
-      <origin xyz="0.15 0.034 0.5" rpy="1.570796 0 1.570796"/>
+      <!--<origin xyz="0.15 0.034 0.5" rpy="1.570796 0 1.570796"/> -->
+      <origin xyz="-0.1 0 0.6" rpy="0 0 1.570796"/>
       <mass value="${m_wingsail}"/>
       <inertia ixx="0.78628153" ixy="-0.00004262" ixz="-0.00044123" iyy="0.32623116" iyz="-0.05493911" izz="0.46187925"/>
     </inertial>
     <visual>
-      <origin xyz="-0.025 -0.015 0" rpy="0 0 0"/>
+      <origin xyz="0.05 0.040 0" rpy="0 0 3.14159"/>
+      <!--<origin xyz="-0.025 -0.015 0" rpy="0 0 0"/> -->
       <geometry>
         <mesh filename="package://mrg_modimoop_description/models/mrg_modimoop_base/mainsail/mainsail.STL" scale="${mesh_scale}"/>
@@ -71,5 +73,5 @@
     </visual>
     <collision name="wingsail_collision">
-      <origin xyz="0.15 0.03 0.675" rpy="0 0 0"/>
+      <origin xyz="-0.1 0.0 0.675" rpy="0 0 0"/>
       <geometry>
         <!-- chord, thickness, height (meters) -->
@@ -80,10 +82,10 @@
   <link name="backwing">
     <inertial>
-      <origin xyz="0.025 0.02 0.2" rpy="1.570796 0 1.570796"/>
+      <origin xyz="-0.035 0.0 0.25" rpy="1.570796 0 1.570796"/>
       <mass value="${m_backwing}"/>
       <inertia ixx="0.00415255" ixy="0.00000002" ixz="0" iyy="0.00011550" iyz="-0.00000140" izz="0.00405022"/>
     </inertial>
     <visual>
-      <origin xyz="-1.3 0.015 -0.5" rpy="1.570796 0 1.570796"/>
+      <origin xyz="1.3 0.0 -0.5" rpy="1.570796 0 -1.570796"/>
       <geometry>
         <mesh filename="package://mrg_modimoop_description/models/mrg_modimoop_base/tailwing/tailwing.STL" scale="${mesh_scale}"/>
@@ -92,5 +94,5 @@
     </visual>
     <collision name="backwing_collision">
-      <origin xyz="0.07 0.03 0.25" rpy="0 0 0"/>
+      <origin xyz="-0.05 0.0 0.25" rpy="0 0 0"/>
       <geometry>
         <!-- chord, thickness, height (meters) -->
@@ -102,10 +104,10 @@
   <link name="rudder">
     <inertial>
-      <origin xyz="0 0.08 -0.08" rpy="0 0 0"/>
+      <origin xyz="-0.074 0 -0.074" rpy="0 0 0"/>
       <mass value="${m_rudder}"/>
       <inertia ixx="0.00323999" ixy="0.00000021" ixz="0.00000004" iyy="0.00089298" iyz="0.00069153" izz="0.00234885"/>
     </inertial>
     <visual>
-      <origin xyz="0 0 0" rpy="0 1.570796 0"/>
+      <origin xyz="0 0 0" rpy="-1.570796 1.570796 0"/>
       <geometry>
         <mesh filename="package://mrg_modimoop_description/models/mrg_modimoop_base/rudder/rudder.STL" scale="${mesh_scale}"/>
@@ -114,5 +116,5 @@
     </visual>
     <collision name="rudder_collision">
-      <origin xyz="0 0.07 -0.075" rpy="1.570796 1.570796 0"/>
+      <origin xyz="-0.074 0 -0.074" rpy="0 1.570796 0"/>
       <geometry>
         <!-- length (fore-aft), thickness, height (meters) -->
@@ -125,5 +127,5 @@
     <inertial>
       <!-- Set the CoM where you expect the keel COM; adjust for your CAD --> <!-- 0.175 -0.55 0.1 -->
-      <origin xyz="0 0 0" rpy="0 0 0"/>
+      <origin xyz="0.0 0.575 -0.55" rpy="0 0 0"/>
       <mass value="${m_keel}"/>
       <inertia ixx="${m_keel*0.016}" ixy="0.0" ixz="0.0" iyy="${m_keel*0.016}" iyz="0.0" izz="${m_keel*0.016}"/>
@@ -132,5 +134,5 @@
     <visual>
       <!-- Align to plate’s CAD frame relative to keel link frame -->
-      <origin xyz="0 0 0" rpy="1.570796 0 3.14159"/>
+      <origin xyz="0.57 0.6025 0" rpy="1.570796 0 -1.570796"/>
       <geometry>
         <mesh filename="package://mrg_modimoop_description/models/mrg_modimoop_base/keel/keel.STL" scale="${mesh_scale}"/>
@@ -140,5 +142,5 @@
     <!-- Plate collision -->
     <collision name="keel_plate_collision">
-      <origin xyz="0.175 -0.55 0.3" rpy="0 0 1.570796"/>
+      <origin xyz="0.0 0.6025 -0.55" rpy="0 0 0"/>
       <geometry>
         <!-- chord, thickness, span (meters) — tune -->
@@ -148,5 +150,5 @@
     <!-- Bulb collision -->
     <collision name="keel_bulb_collision">
-      <origin xyz="0.175 -0.565 -0.08" rpy="1.570796 0 0"/>
+      <origin xyz="0.0 0.6025 -0.79" rpy="1.570796 0 1.570796"/>
       <geometry>
         <!-- length is along cylinder Z axis in its collision frame -->
@@ -168,5 +170,5 @@
     <parent link="hull"/>
     <child link="wingsail"/>
-    <origin xyz="0.2 -0.65 0.65" rpy="0 0 1.570796"/>
+    <origin xyz="0.3 -0.545 0.65" rpy="0 0 0"/>
     <axis xyz="0 0 1"/>
     <dynamics damping="0.2" friction="0.0"/>
@@ -176,5 +178,5 @@
     <parent link="wingsail"/>
     <child link="backwing_hinge"/>
-    <origin xyz="0.45 0.0125 0.4" rpy="0 0 0"/>
+    <origin xyz="-0.8 0.0 0.4" rpy="0 0 0"/>
   </joint>
   <joint name="backwing_joint" type="continuous">
@@ -190,5 +192,5 @@
     <parent link="hull"/>
     <child link="rudder"/>
-    <origin xyz="0.175 -0.3 0.3" rpy="0 0 0"/>
+    <origin xyz="-0.1 -0.545 0.3" rpy="0 0 0"/>
     <axis xyz="0 0 1"/>
     <dynamics damping="0.1" friction="0.0"/>
@@ -211,14 +213,14 @@
     <parent link="hull"/>
     <child link="rudder_rod"/>
-    <origin xyz="0.175 -0.3 0.3" rpy="0 0 0"/>
+    <origin xyz="-0.1 -0.545 0.3" rpy="0 0 0"/>
   </joint>
   <link name="wingsail_rod">
     <inertial>
-      <origin xyz="0 0 0" rpy="0 0 0"/>
+      <origin xyz="0.105 -0.1025 0" rpy="0 0 0"/>
       <mass value="${rod_mass}"/>
       <inertia ixx="1e-6" ixy="0" ixz="0" iyy="1e-6" iyz="0" izz="1e-6"/>
     </inertial>
     <visual>
-      <origin xyz="0 0.01 0" rpy="0 0 0"/>
+      <origin xyz="0.105 -0.1025 0" rpy="0 0 0"/>
       <geometry>
         <cylinder radius="${wingsail_rod_radius}" length="0.40"/>
@@ -234,5 +236,5 @@
   <link name="backwing_rod_top">
     <inertial>
-      <origin xyz="0 0 0" rpy="0 0 0"/>
+      <origin xyz="0 0 0.73" rpy="0 0 0"/>
       <mass value="${rod_mass}"/>
       <inertia ixx="1e-6" ixy="0" ixz="0" iyy="1e-6" iyz="0" izz="1e-6"/>
@@ -240,7 +242,7 @@
     <visual>
       <!-- Rotate cylinder so it runs along X -->
-      <origin xyz="-0.1 0.008 0.73" rpy="0 1.570796 0"/>
-      <geometry>
-        <cylinder radius="${backwing_rod_radius}" length="0.625"/>
+      <origin xyz="-0.5 -0.025 0.73" rpy="0 1.570796 0"/>
+      <geometry>
+        <cylinder radius="${backwing_rod_radius}" length="1.2"/>
       </geometry>
       <material name="Black"/>
@@ -249,12 +251,12 @@
   <link name="backwing_rod_bottom">
     <inertial>
-      <origin xyz="0 0 0" rpy="0 0 0"/>
+      <origin xyz="0 0 0.32" rpy="0 0 0"/>
       <mass value="${rod_mass}"/>
       <inertia ixx="1e-6" ixy="0" ixz="0" iyy="1e-6" iyz="0" izz="1e-6"/>
     </inertial>
     <visual>
-      <origin xyz="-0.1 0.008 0.32" rpy="0 1.570796 0"/>
-      <geometry>
-        <cylinder radius="${backwing_rod_radius}" length="0.625"/>
+      <origin xyz="-0.5 -0.025 0.32" rpy="0 1.570796 0"/>
+      <geometry>
+        <cylinder radius="${backwing_rod_radius}" length="1.2"/>
       </geometry>
       <material name="Black"/>
@@ -310,7 +312,7 @@
           <area>0.17</area>
           <fluid_density>1.225</fluid_density>
-          <forward>-1 0 0</forward>
+          <forward>1 0 0</forward>
           <upward>0 1 0</upward>
-          <cp>0.15 0.034 0.5</cp>
+          <cp>-0.1 0 0.6</cp>
           <link_name>wingsail</link_name>
           <radial_symmetry>1</radial_symmetry>
@@ -326,7 +328,7 @@
           <area>0.05</area>
           <fluid_density>1.225</fluid_density>
-          <forward>-1 0 0</forward>
+          <forward>1 0 0</forward>
           <upward>0 1 0</upward>
-          <cp>0.025 0.02 0.2</cp>
+          <cp>-0.035 0.0 0.25</cp>
           <link_name>backwing</link_name>
           <radial_symmetry>1</radial_symmetry>
@@ -342,7 +344,7 @@
           <area>0.17</area>
           <fluid_density>1000</fluid_density>
-          <forward>0 -1 0</forward>
-          <upward>1 0 0</upward>
-          <cp>0.175 -0.55 0.1</cp>
+          <forward>1 0 0</forward>
+          <upward>0 1 0</upward>
+          <cp>0.0 0.575 -0.55</cp>
           <link_name>keel</link_name>
           <radial_symmetry>1</radial_symmetry>
@@ -358,7 +360,7 @@
           <area>0.12</area>
           <fluid_density>1000</fluid_density>
-          <forward>0 -1 0</forward>
-          <upward>1 0 0</upward>
-          <cp>0 0.08 -0.08</cp>
+          <forward>1 0 0</forward>
+          <upward>0 1 0</upward>
+          <cp>-0.074 0 -0.074</cp>
           <link_name>rudder</link_name>
           <radial_symmetry>1</radial_symmetry>

Commit message: Fixed sensor yaws to match the world frame as I expect; hardcoded fixes are no longer present in the localization class in the controls package

File: mrg_modimoop_description/urdf/mrg_modimoop.urdf.xacro (robot description, xacro)
@@ -43,5 +43,5 @@
     </inertial>
     <visual>
-      <origin xyz="-0.41 -0.725 0" rpy="1.570796 0 1.570796"/>
+      <origin xyz="-0.41 -0.725 0" rpy="${pi/2} 0 ${pi/2}"/>
       <geometry>
         <mesh filename="package://mrg_modimoop_description/models/mrg_modimoop_base/hull/hull.STL" scale="${mesh_scale}"/>
@@ -50,5 +50,5 @@
     </visual>
     <collision name="hull_collision">
-      <origin xyz="0.178 -0.55 0.45" rpy="0 0 3.14159"/>
+      <origin xyz="0.178 -0.55 0.45" rpy="0 0 ${pi}"/>
       <geometry>
         <box size="1.125 0.35 0.25"/>
@@ -60,10 +60,10 @@
     <inertial>
       <!--<origin xyz="0.15 0.034 0.5" rpy="1.570796 0 1.570796"/> -->
-      <origin xyz="-0.1 0 0.6" rpy="0 0 1.570796"/>
+      <origin xyz="-0.1 0 0.6" rpy="0 0 ${pi/2}"/>
       <mass value="${m_wingsail}"/>
       <inertia ixx="0.78628153" ixy="-0.00004262" ixz="-0.00044123" iyy="0.32623116" iyz="-0.05493911" izz="0.46187925"/>
     </inertial>
     <visual>
-      <origin xyz="0.05 0.040 0" rpy="0 0 3.14159"/>
+      <origin xyz="0.05 0.040 0" rpy="0 0 ${pi}"/>
       <!--<origin xyz="-0.025 -0.015 0" rpy="0 0 0"/> -->
       <geometry>
@@ -82,10 +82,10 @@
   <link name="backwing">
     <inertial>
-      <origin xyz="-0.035 0.0 0.25" rpy="1.570796 0 1.570796"/>
+      <origin xyz="-0.035 0.0 0.25" rpy="${pi/2} 0 ${pi/2}"/>
       <mass value="${m_backwing}"/>
       <inertia ixx="0.00415255" ixy="0.00000002" ixz="0" iyy="0.00011550" iyz="-0.00000140" izz="0.00405022"/>
     </inertial>
     <visual>
-      <origin xyz="1.3 0.0 -0.5" rpy="1.570796 0 -1.570796"/>
+      <origin xyz="1.3 0.0 -0.5" rpy="${pi/2} 0 -${pi/2}"/>
       <geometry>
         <mesh filename="package://mrg_modimoop_description/models/mrg_modimoop_base/tailwing/tailwing.STL" scale="${mesh_scale}"/>
@@ -109,5 +109,5 @@
     </inertial>
     <visual>
-      <origin xyz="0 0 0" rpy="-1.570796 1.570796 0"/>
+      <origin xyz="0 0 0" rpy="-${pi/2} ${pi/2} 0"/>
       <geometry>
         <mesh filename="package://mrg_modimoop_description/models/mrg_modimoop_base/rudder/rudder.STL" scale="${mesh_scale}"/>
@@ -116,5 +116,5 @@
     </visual>
     <collision name="rudder_collision">
-      <origin xyz="-0.074 0 -0.074" rpy="0 1.570796 0"/>
+      <origin xyz="-0.074 0 -0.074" rpy="0 ${pi/2} 0"/>
       <geometry>
         <!-- length (fore-aft), thickness, height (meters) -->
@@ -134,5 +134,5 @@
     <visual>
       <!-- Align to plate’s CAD frame relative to keel link frame -->
-      <origin xyz="0.57 0.6025 0" rpy="1.570796 0 -1.570796"/>
+      <origin xyz="0.57 0.6025 0" rpy="${pi/2} 0 -${pi/2}"/>
       <geometry>
         <mesh filename="package://mrg_modimoop_description/models/mrg_modimoop_base/keel/keel.STL" scale="${mesh_scale}"/>
@@ -150,5 +150,5 @@
     <!-- Bulb collision -->
     <collision name="keel_bulb_collision">
-      <origin xyz="0.0 0.6025 -0.79" rpy="1.570796 0 1.570796"/>
+      <origin xyz="0.0 0.6025 -0.79" rpy="${pi/2} 0 ${pi/2}"/>
       <geometry>
         <!-- length is along cylinder Z axis in its collision frame -->
@@ -172,5 +172,5 @@
     <origin xyz="0.3 -0.545 0.65" rpy="0 0 0"/>
     <axis xyz="0 0 1"/>
-    <dynamics damping="0.2" friction="0.0"/>
+    <dynamics damping="2.5" friction="0.45"/>
   </joint>
   <link name="backwing_hinge"/>
@@ -186,5 +186,5 @@
     <!-- coaxial -->
     <axis xyz="0 0 1"/>
-    <dynamics damping="0.05" friction="0.0"/>
+    <dynamics damping="0.2" friction="0.35"/>
   </joint>
   <!-- Rudder rotates around Z for yaw -->
@@ -194,5 +194,5 @@
     <origin xyz="-0.1 -0.545 0.3" rpy="0 0 0"/>
     <axis xyz="0 0 1"/>
-    <dynamics damping="0.1" friction="0.0"/>
+    <dynamics damping="0.2" friction="0.35"/>
   </joint>
   <link name = "rudder_rod">
@@ -280,5 +280,4 @@
     <parent link="hull"/>
     <child link="imu_link"/>
-    <!-- put IMU near your hull CG -->
     <origin xyz="0.175 -0.55 0.45" rpy="0 0 0"/>
   </joint>
@@ -294,5 +293,5 @@
     <parent link="hull"/>
     <child link="anemometer_link"/>
-    <origin xyz="0.25 -0.55 1.00" rpy="0 0 0"/>
+    <origin xyz="0.25 -0.55 1.00" rpy="0 0 ${pi}"/>
   </joint>
   <link name="mag_link"/>
@@ -343,5 +342,5 @@
           <cda>0.63662</cda>
           <area>0.17</area>
-          <fluid_density>1000</fluid_density>
+          <fluid_density>1025</fluid_density>
           <forward>1 0 0</forward>
           <upward>0 1 0</upward>
@@ -354,10 +353,10 @@
             filename="asv_sim2-foil-lift-drag-system">
           <a0>0.0</a0>
-          <cla>6.2832</cla>
+          <cla>5.0</cla>
           <alpha_stall>0.1592</alpha_stall>
           <cla_stall>-0.7083</cla_stall>
           <cda>0.63662</cda>
-          <area>0.12</area>
-          <fluid_density>1000</fluid_density>
+          <area>0.02322576</area>
+          <fluid_density>1025</fluid_density>
           <forward>1 0 0</forward>
           <upward>0 1 0</upward>
@@ -384,5 +383,5 @@
         </plugin>
   </gazebo>
-    <!-- ===================== -->
+  <!-- ===================== -->
   <!-- Gazebo sensors        -->
   <!-- ===================== -->
@@ -395,4 +394,5 @@
       <topic>/modimoop/imu</topic>
       <gz_frame_id>imu_link</gz_frame_id>
+      <pose>0 0 0 0 -1.570796327</pose>
       <imu>
         <angular_velocity>
@@ -421,4 +421,5 @@
       <topic>anemometer</topic>
       <gz_frame_id>aneomometer_link</gz_frame_id>
+      <pose>0 0 0 0 0 0</pose>
       <gz:anemometer>
          <!-- <noise type="gaussian">
@@ -436,4 +437,5 @@
       <topic>/modimoop/navsat</topic>
       <gz_frame_id>gps_link</gz_frame_id>
+      <pose>0 0 0 0 0 -1.570796327</pose>
       <visualize>0</visualize>
     </sensor>
@@ -447,4 +449,5 @@
       <topic>/modimoop/mag</topic>
       <gz_frame_id>mag_link</gz_frame_id>
+      <pose>0 0 0 0 0 -1.570796327</pose>
       <magnetometer/>
     </sensor>
@@ -465,5 +468,4 @@
       <joint_name>wingsail_joint</joint_name>
       <topic>/modimoop/cmd/wingsail_pos</topic>
-      <!-- optional PID knobs depending on version; start without -->
     </plugin>
     <plugin filename="gz-sim-joint-position-controller-system"

Commit message: Updated MRG modimoop

File: mrg_modimoop_description/urdf/mrg_modimoop.urdf.xacro (robot description, xacro)
@@ -172,5 +172,5 @@
     <origin xyz="0.3 -0.545 0.65" rpy="0 0 0"/>
     <axis xyz="0 0 1"/>
-    <dynamics damping="2.5" friction="0.45"/>
+    <dynamics damping="0.2" friction="0.05"/>
   </joint>
   <link name="backwing_hinge"/>
@@ -186,5 +186,5 @@
     <!-- coaxial -->
     <axis xyz="0 0 1"/>
-    <dynamics damping="0.2" friction="0.35"/>
+    <dynamics damping="0.2" friction="0.05"/>
   </joint>
   <!-- Rudder rotates around Z for yaw -->
@@ -194,5 +194,5 @@
     <origin xyz="-0.1 -0.545 0.3" rpy="0 0 0"/>
     <axis xyz="0 0 1"/>
-    <dynamics damping="0.2" friction="0.35"/>
+    <dynamics damping="0.2" friction="0.05"/>
   </joint>
   <link name = "rudder_rod">
@@ -313,5 +313,6 @@
           <forward>1 0 0</forward>
           <upward>0 1 0</upward>
-          <cp>-0.1 0 0.6</cp>
+          <!--<cp>-0.1 0 0.6</cp>-->
+          <cp>0.2, -0.545, 1.25</cp> <!-- Defined as parent frame offset + CoM offset -->
           <link_name>wingsail</link_name>
           <radial_symmetry>1</radial_symmetry>
@@ -329,5 +330,6 @@
           <forward>1 0 0</forward>
           <upward>0 1 0</upward>
-          <cp>-0.035 0.0 0.25</cp>
+          <!--<cp>-0.035 0.0 0.25</cp>-->
+          <cp>-0.035 0.0 0.25</cp> <!-- Defined as parent frame offset + CoM offset -->
           <link_name>backwing</link_name>
           <radial_symmetry>1</radial_symmetry>
@@ -345,5 +347,6 @@
           <forward>1 0 0</forward>
           <upward>0 1 0</upward>
-          <cp>0.0 0.575 -0.55</cp>
+          <!--<cp>0.0 0.575 -0.55</cp>-->
+          <cp>0.175 -0.575 0.15</cp> <!-- Defined as parent frame offset + CoM offset -->
           <link_name>keel</link_name>
           <radial_symmetry>1</radial_symmetry>
@@ -361,5 +364,6 @@
           <forward>1 0 0</forward>
           <upward>0 1 0</upward>
-          <cp>-0.074 0 -0.074</cp>
+          <!--<cp>-0.074 0 -0.074</cp>-->
+          <cp>-0.174 -0.545 0.226</cp> <!-- Defined as parent frame offset + CoM offset -->
           <link_name>rudder</link_name>
           <radial_symmetry>1</radial_symmetry>
