Commit message: Updated the URDF to use the SolidWorks to URDF Pipeline URDF file. Also updated the meshes for all visuals, and updated the collision meshes. This consolidated the hull and keel into a single link, unlike the previous version. So far, this has resulted in more correct hydrodynamic behavior. There are now several options for collision meshes for the hull. A three-collision component, which is very low fidelity, can be used in place of a better collision mesh if performance isn't particularly important. Otherwise, there are meshes with 100, 200, 300, 500, 1000, and the original mesh that can be chosen for collision.

File: mrg_modimoop_description/urdf/mrg_modimoop.urdf.xacro (robot description, xacro)
@@ -1,394 +1,239 @@
-<?xml version="1.0" ?>
-<!-- =================================================================================== -->
-<!-- |    This document was autogenerated by xacro from /root/mrg_ws/install/share/mrg_modimoop/urdf/mrg_modimoop.urdf.xacro | -->
-<!-- |    EDITING THIS FILE BY HAND IS NOT RECOMMENDED                                 | -->
-<!-- =================================================================================== -->
-<!-- Basic MODIMOOP description -->
+<?xml version='1.0' encoding='UTF-8'?>
 <robot xmlns:xacro="http://www.ros.org/wiki/xacro" xmlns:gz="http://gazebosim.org/schema" name="MODIMOOP">
-  <!-- ===================== -->
-  <!-- Common parameters     -->
-  <!-- ===================== -->
-  <xacro:property name="mesh_scale" value="0.001 0.001 0.001"/>
-  <xacro:property name="backwing_mesh_scale" value="0.0004 0.0004 0.0004"/>
-  <!-- Rough masses (kg). Replace with measured values -->
-  <xacro:property name="m_hull"     value="22.83"/>
-  <xacro:property name="m_keel"     value="0.01"/>        <!-- total for keel (plate+bulb) if single link -->
-  <xacro:property name="m_wingsail" value="4.44"/>
-  <xacro:property name="m_rudder"   value="0.34"/>
-  <xacro:property name="m_backwing" value="0.17"/>
-  <xacro:property name="rudder_rod_radius" value="0.0045"/>
-  <xacro:property name="wingsail_rod_radius" value="0.01"/>
-  <xacro:property name="backwing_rod_radius" value="0.008"/>
-  <xacro:property name="rod_mass" value="0.001"/>
-  <!-- Simple diagonal inertias (kg·m²). Replace with real inertias -->
-  <xacro:property name="I_small" value="0.02"/>
-  <!-- Materials -->
-  <material name="Grey"><color rgba="0.6 0.6 0.6 1.0"/></material>
-  <material name="Blue"><color rgba="0.2 0.4 0.8 1.0"/></material>
-  <material name="Red"><color rgba="0.8 0.2 0.2 1.0"/></material>
-  <material name="Black"><color rgba="0.05 0.05 0.05 1.0"/></material>
-  <material name="Pink"><color rgba="1.0 0.2 0.6 1.0"/></material>
-  <!-- ===================== -->
-  <!-- Links                 -->
-  <!-- ===================== -->
-  <!-- Hull is the base -->
-  <link name="hull">
+  <xacro:arg name="model_name" default="none_mrg_modimoop"/>
+  <xacro:arg name="keel_cp" default="-0.633 0 -0.351"/>
+  <link name="hull_link">
     <inertial>
-      <!--<origin xyz="0 0.75915 -1.33874" rpy="0 0 0"/>-->
-      <origin xyz="0.175 -0.55 0.15" rpy="0 0 1.570796"/>
-      <!--<origin xyz="0.175 -1.1 0.575" rpy="0 0 0"/>-->
-      <!--<origin xyz="0.175 -0.34085 0.575" rpy="0 0 0"/>-->
-      <mass value="${m_hull}"/>
-      <inertia ixx="3.70506895" ixy="-0.00022839" ixz="-0.00008461" iyy="0.96696277" iyz="-0.64724529" izz="2.83543540"/>
+      <origin xyz="-0.633 0 -0.351" rpy="0 0 0"/>
+      <mass value="22.44"/>
+      <inertia ixx="1.96" ixy="0" ixz="-0.529" iyy="2.85" iyz="-0.001" izz="0.99"/>
     </inertial>
     <visual>
-      <origin xyz="-0.41 -0.725 0" rpy="${pi/2} 0 ${pi/2}"/>
-      <geometry>
-        <mesh filename="package://mrg_modimoop_description/models/mrg_modimoop_base/hull/hull.STL" scale="${mesh_scale}"/>
-      </geometry>
-      <material name="Pink"/>
+      <origin xyz="0 0 0" rpy="0 0 0"/>
+      <geometry>
+        <mesh filename="package://mrg_modimoop_description/models/meshes/hull_link.STL"/>
+      </geometry>
+      <material name="">
+        <color rgba="1 1 1 1"/>
+      </material>
     </visual>
+    <!-- Do not use the hull_hydro_100 mesh, it gives poor results. Generally, 200+ gives good hydrodynamic results but slow downs happen quickly -->
     <collision name="hull_collision">
-      <origin xyz="0.178 -0.55 0.45" rpy="0 0 ${pi}"/>
-      <geometry>
-        <box size="1.125 0.35 0.25"/>
-      </geometry>
-    </collision>
+      <origin xyz="0 0 0" rpy="0 0 0"/>
+      <geometry>
+        <mesh filename="package://mrg_modimoop_description/models/meshes/hull_hydro_200.STL"/>
+      </geometry>
+    </collision>
+    <!-- Consider using this collision where perfect accuracy is fine initially (i.e. training models or something) -->
+    <!--
+    <collision name="hull_hydro_collision">
+      <origin xyz="0.0 0 0" rpy="0 0 0"/>
+      <geometry>
+        <mesh filename="package://mrg_modimoop_description/models/meshes/hull_wedge_box.STL"/>
+      </geometry>
+    </collision>
+    <collision name="keel_plate_collision">
+      <origin xyz="-0.575 0 -0.46" rpy="0 0 0"/>
+      <geometry>
+        <box size="0.10 0.0125 0.48"/>
+      </geometry>
+    </collision>
+    <collision name="keel_ballast_collision">
+      <origin xyz="-0.6 0 -0.65" rpy="0 0 0"/>
+      <geometry>
+        <box size="0.325 0.09 0.09"/>
+      </geometry>
+    </collision>
+    -->
   </link>
-  <!-- Wingsail (revolute about vertical axis for trim) -->
-  <link name="wingsail">
+  <link name="wingsail_link">
     <inertial>
-      <!--<origin xyz="0.15 0.034 0.5" rpy="1.570796 0 1.570796"/> -->
-      <origin xyz="-0.1 0 0.6" rpy="0 0 ${pi/2}"/>
-      <mass value="${m_wingsail}"/>
-      <inertia ixx="0.78628153" ixy="-0.00004262" ixz="-0.00044123" iyy="0.32623116" iyz="-0.05493911" izz="0.46187925"/>
+      <origin xyz="0 0 0.559" rpy="0 0 0"/>
+      <mass value="4.181"/>
+      <inertia ixx="0.441" ixy="0" ixz="-0.029" iyy="0.668" iyz="0" izz="0.23"/>
     </inertial>
     <visual>
-      <origin xyz="0.05 0.040 0" rpy="0 0 ${pi}"/>
-      <!--<origin xyz="-0.025 -0.015 0" rpy="0 0 0"/> -->
-      <geometry>
-        <mesh filename="package://mrg_modimoop_description/models/mrg_modimoop_base/mainsail/mainsail.STL" scale="${mesh_scale}"/>
-      </geometry>
-      <material name="Pink"/>
+      <origin xyz="0 0 0" rpy="0 0 0"/>
+      <geometry>
+        <mesh filename="package://mrg_modimoop_description/models/meshes/wingsail_link.STL"/>
+      </geometry>
+      <material name="">
+        <color rgba="1 1 1 1"/>
+      </material>
     </visual>
     <collision name="wingsail_collision">
-      <origin xyz="-0.1 0.0 0.675" rpy="0 0 0"/>
-      <geometry>
-        <!-- chord, thickness, height (meters) -->
-        <box size="0.30 0.04 1.32"/>
+      <origin xyz="0 0 0" rpy="0 0 0"/>
+      <geometry>
+        <mesh filename="package://mrg_modimoop_description/models/meshes/wingsail_link.STL"/>
       </geometry>
     </collision>
   </link>
-  <link name="backwing">
+  <joint name="wingsail_joint" type="continuous">
+    <origin xyz="-0.55 0 0" rpy="0 0 0"/>
+    <parent link="hull_link"/>
+    <child link="wingsail_link"/>
+    <axis xyz="0 0 1"/>
+    <dynamics damping="0.2" friction="0.05"/>
+  </joint>
+  <link name="tailwing_link">
     <inertial>
-      <origin xyz="-0.035 0.0 0.25" rpy="${pi/2} 0 ${pi/2}"/>
-      <mass value="${m_backwing}"/>
-      <inertia ixx="0.00415255" ixy="0.00000002" ixz="0" iyy="0.00011550" iyz="-0.00000140" izz="0.00405022"/>
+      <origin xyz="-0.017 0 -0.016" rpy="0 0 0"/>
+      <mass value="0.201"/>
+      <inertia ixx="0.006" ixy="0" ixz="0" iyy="0.006" iyz="0" izz="0.00001"/>
     </inertial>
     <visual>
-      <origin xyz="1.3 0.0 -0.5" rpy="${pi/2} 0 -${pi/2}"/>
-      <geometry>
-        <mesh filename="package://mrg_modimoop_description/models/mrg_modimoop_base/tailwing/tailwing.STL" scale="${mesh_scale}"/>
-      </geometry>
-      <material name="Pink"/>
+      <origin xyz="0 0 0" rpy="0 0 0"/>
+      <geometry>
+        <mesh filename="package://mrg_modimoop_description/models/meshes/tailwing_link.STL"/>
+      </geometry>
+      <material name="">
+        <color rgba="1 1 1 1"/>
+      </material>
     </visual>
-    <collision name="backwing_collision">
-      <origin xyz="-0.05 0.0 0.25" rpy="0 0 0"/>
-      <geometry>
-        <!-- chord, thickness, height (meters) -->
-        <box size="0.11 0.02 0.55"/>
+    <collision name="tailwing_collision">
+      <origin xyz="0 0 0" rpy="0 0 0"/>
+      <geometry>
+        <mesh filename="package://mrg_modimoop_description/models/meshes/tailwing_link.STL"/>
       </geometry>
     </collision>
   </link>
-  <!-- Rudder (revolute about vertical axis) -->
-  <link name="rudder">
+  <joint name="tailwing_joint" type="revolute">
+    <origin xyz="-0.7485 0 0.73529" rpy="0 0 0"/>
+    <parent link="wingsail_link"/>
+    <child link="tailwing_link"/>
+    <axis xyz="0 0 -1"/>
+    <limit lower="-0.785" upper="0.785" effort="5.0" velocity="1.0"/>
+    <dynamics damping="0.2" friction="0.05"/>
+  </joint>
+  <link name="rudder_link">
     <inertial>
-      <origin xyz="-0.074 0 -0.074" rpy="0 0 0"/>
-      <mass value="${m_rudder}"/>
-      <inertia ixx="0.00323999" ixy="0.00000021" ixz="0.00000004" iyy="0.00089298" iyz="0.00069153" izz="0.00234885"/>
+      <origin xyz="0 0 0" rpy="0 0 0"/>
+      <mass value="0.34"/>
+      <inertia ixx="0.001" ixy="0" ixz="0" iyy="0.001" iyz="0" izz="0.001"/>
     </inertial>
     <visual>
-      <origin xyz="0 0 0" rpy="-${pi/2} ${pi/2} 0"/>
-      <geometry>
-        <mesh filename="package://mrg_modimoop_description/models/mrg_modimoop_base/rudder/rudder.STL" scale="${mesh_scale}"/>
-      </geometry>
-      <material name="Black"/>
+      <origin xyz="0 0 0" rpy="0 0 0"/>
+      <geometry>
+        <mesh filename="package://mrg_modimoop_description/models/meshes/rudder_link.STL"/>
+      </geometry>
+      <material name="">
+        <color rgba="1 1 1 1"/>
+      </material>
     </visual>
     <collision name="rudder_collision">
-      <origin xyz="-0.074 0 -0.074" rpy="0 ${pi/2} 0"/>
-      <geometry>
-        <!-- length (fore-aft), thickness, height (meters) -->
-        <box size="0.15 0.01 0.15"/>
+      <origin xyz="0 0 0" rpy="0 0 0"/>
+      <geometry>
+        <mesh filename="package://mrg_modimoop_description/models/meshes/rudder_link.STL"/>
       </geometry>
     </collision>
   </link>
-  <!-- Keel as a single link with two mesh components (plate + bulb) -->
-  <link name="keel">
-    <inertial>
-      <!-- Set the CoM where you expect the keel COM; adjust for your CAD --> <!-- 0.175 -0.55 0.1 -->
-      <origin xyz="0.0 0.575 -0.55" rpy="0 0 0"/>
-      <mass value="${m_keel}"/>
-      <inertia ixx="${m_keel*0.016}" ixy="0.0" ixz="0.0" iyy="${m_keel*0.016}" iyz="0.0" izz="${m_keel*0.016}"/>
-    </inertial>
-    <!-- Keel visual -->
-    <visual>
-      <!-- Align to plate’s CAD frame relative to keel link frame -->
-      <origin xyz="0.57 0.6025 0" rpy="${pi/2} 0 -${pi/2}"/>
-      <geometry>
-        <mesh filename="package://mrg_modimoop_description/models/mrg_modimoop_base/keel/keel.STL" scale="${mesh_scale}"/>
-      </geometry>
-      <material name="Grey"/>
-    </visual>
-    <!-- Plate collision -->
-    <collision name="keel_plate_collision">
-      <origin xyz="0.0 0.6025 -0.55" rpy="0 0 0"/>
-      <geometry>
-        <!-- chord, thickness, span (meters) — tune -->
-        <box size="0.175 0.0125 0.70"/>
-      </geometry>
-    </collision>
-    <!-- Bulb collision -->
-    <collision name="keel_bulb_collision">
-      <origin xyz="0.0 0.6025 -0.79" rpy="${pi/2} 0 ${pi/2}"/>
-      <geometry>
-        <!-- length is along cylinder Z axis in its collision frame -->
-        <cylinder length="0.325" radius="0.045"/>
-      </geometry>
-    </collision>
-  </link>
-  <!-- ===================== -->
-  <!-- Joints                -->
-  <!-- ===================== -->
-  <!-- Keel fixed to hull -->
-  <joint name="keel_mount" type="fixed">
-    <parent link="hull"/>
-    <child link="keel"/>
-    <origin xyz="0.175 -1.15 0.7" rpy="0 0 0"/>
-  </joint>
-  <!-- Wingsail rotates around Z (trim). Limit range ±90° by default -->
-  <joint name="wingsail_joint" type="continuous">
-    <parent link="hull"/>
-    <child link="wingsail"/>
-    <origin xyz="0.3 -0.545 0.65" rpy="0 0 0"/>
+  <joint name="rudder_joint" type="revolute">
+    <origin xyz="-0.850348439870171 0 -0.25961" rpy="0 0 0"/>
+    <parent link="hull_link"/>
+    <child link="rudder_link"/>
     <axis xyz="0 0 1"/>
+    <limit lower="-0.785" upper="0.785" effort="5.0" velocity="1.0"/>
     <dynamics damping="0.2" friction="0.05"/>
   </joint>
-  <link name="backwing_hinge"/>
-  <joint name="backwing_hinge_joint" type="fixed">
-    <parent link="wingsail"/>
-    <child link="backwing_hinge"/>
-    <origin xyz="-0.8 0.0 0.4" rpy="0 0 0"/>
-  </joint>
-  <joint name="backwing_joint" type="continuous">
-    <parent link="backwing_hinge"/>
-    <child link="backwing"/>
-    <origin xyz="0 0 0" rpy="0 0 0"/>
-    <!-- coaxial -->
-    <axis xyz="0 0 1"/>
-    <dynamics damping="0.2" friction="0.05"/>
-  </joint>
-  <!-- Rudder rotates around Z for yaw -->
-  <joint name="rudder_joint" type="continuous">
-    <parent link="hull"/>
-    <child link="rudder"/>
-    <origin xyz="-0.1 -0.545 0.3" rpy="0 0 0"/>
-    <axis xyz="0 0 1"/>
-    <dynamics damping="0.2" friction="0.05"/>
-  </joint>
-  <link name = "rudder_rod">
-    <inertial>
-      <origin xyz="0 0 0" rpy = "0 0 0"/>
-      <mass value="${rod_mass}"/>
-      <inertia ixx="1e-6" ixy="0" ixz="0" iyy="1e-6" iyz="0" izz="1e-6"/>
-    </inertial>
-    <visual>
-      <origin xyz="0 0 0" rpy="0 0 0"/>
-      <geometry>
-        <cylinder radius="${rudder_rod_radius}" length="0.20"/>
-      </geometry>
-      <material name="Black"/>
-    </visual>
-  </link>
-  <joint name="rudder_rod_mount" type="fixed">
-    <parent link="hull"/>
-    <child link="rudder_rod"/>
-    <origin xyz="-0.1 -0.545 0.3" rpy="0 0 0"/>
-  </joint>
-  <link name="wingsail_rod">
-    <inertial>
-      <origin xyz="0.105 -0.1025 0" rpy="0 0 0"/>
-      <mass value="${rod_mass}"/>
-      <inertia ixx="1e-6" ixy="0" ixz="0" iyy="1e-6" iyz="0" izz="1e-6"/>
-    </inertial>
-    <visual>
-      <origin xyz="0.105 -0.1025 0" rpy="0 0 0"/>
-      <geometry>
-        <cylinder radius="${wingsail_rod_radius}" length="0.40"/>
-      </geometry>
-      <material name="Black"/>
-    </visual>
-  </link>
-  <joint name="wingsail_rod_mount" type="fixed">
-    <parent link="hull"/>
-    <child link="wingsail_rod"/>
-    <origin xyz="0.2 -0.65 0.65" rpy="0 0 1.570796"/>
-  </joint>
-  <link name="backwing_rod_top">
-    <inertial>
-      <origin xyz="0 0 0.73" rpy="0 0 0"/>
-      <mass value="${rod_mass}"/>
-      <inertia ixx="1e-6" ixy="0" ixz="0" iyy="1e-6" iyz="0" izz="1e-6"/>
-    </inertial>
-    <visual>
-      <!-- Rotate cylinder so it runs along X -->
-      <origin xyz="-0.5 -0.025 0.73" rpy="0 1.570796 0"/>
-      <geometry>
-        <cylinder radius="${backwing_rod_radius}" length="1.2"/>
-      </geometry>
-      <material name="Black"/>
-    </visual>
-  </link>
-  <link name="backwing_rod_bottom">
-    <inertial>
-      <origin xyz="0 0 0.32" rpy="0 0 0"/>
-      <mass value="${rod_mass}"/>
-      <inertia ixx="1e-6" ixy="0" ixz="0" iyy="1e-6" iyz="0" izz="1e-6"/>
-    </inertial>
-    <visual>
-      <origin xyz="-0.5 -0.025 0.32" rpy="0 1.570796 0"/>
-      <geometry>
-        <cylinder radius="${backwing_rod_radius}" length="1.2"/>
-      </geometry>
-      <material name="Black"/>
-    </visual>
-  </link>
-  <joint name="backwing_rod_top_mount" type="fixed">
-    <parent link="wingsail"/>
-    <child link="backwing_rod_top"/>
-    <origin xyz="0.25 0.02 0.2" rpy="0 0 0"/>
-  </joint>
-  <joint name="backwing_rod_bottom_mount" type="fixed">
-    <parent link="wingsail"/>
-    <child link="backwing_rod_bottom"/>
-    <origin xyz="0.25 0.02 0.05" rpy="0 0 0"/>
-  </joint>
-  <!-- ===================== -->
-  <!-- Sensor frame links    -->
-  <!-- ===================== -->
   <link name="imu_link"/>
   <joint name="imu_mount" type="fixed">
-    <parent link="hull"/>
+    <parent link="hull_link"/>
     <child link="imu_link"/>
-    <origin xyz="0.175 -0.55 0.45" rpy="0 0 0"/>
+    <origin xyz="-0.675 -0.005 -0.2" rpy="0 0 0"/>
   </joint>
   <link name="gps_link"/>
   <joint name="gps_mount" type="fixed">
-    <parent link="hull"/>
+    <parent link="hull_link"/>
     <child link="gps_link"/>
-    <!-- e.g., GPS on deck -->
-    <origin xyz="0.25 -0.55 0.75" rpy="0 0 0"/>
+    <origin xyz="-0.6 -0.005 0.1" rpy="0 0 0"/>
   </joint>
   <link name="anemometer_link"/>
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
Commit message: Fixed an error where the wingsail was being commanded to the zero position constantly; it should not do that

File: mrg_modimoop_description/urdf/mrg_modimoop.urdf.xacro (robot description, xacro)
@@ -103,5 +103,5 @@
     <child link="tailwing_link"/>
     <axis xyz="0 0 -1"/>
-    <limit lower="-0.785" upper="0.785" effort="5.0" velocity="1.0"/>
+    <limit lower="-0.785" upper="0.785" effort="1.0" velocity="0.2"/>
     <dynamics damping="0.2" friction="0.05"/>
   </joint>
@@ -133,5 +133,5 @@
     <child link="rudder_link"/>
     <axis xyz="0 0 1"/>
-    <limit lower="-0.785" upper="0.785" effort="5.0" velocity="1.0"/>
+    <limit lower="-0.785" upper="0.785" effort="1.0" velocity="0.2"/>
     <dynamics damping="0.2" friction="0.05"/>
   </joint>
@@ -357,8 +357,4 @@
   <gazebo>
     <plugin filename="gz-sim-joint-position-controller-system" name="gz::sim::systems::JointPositionController">
-      <joint_name>wingsail_joint</joint_name>
-      <topic>/modimoop/cmd/wingsail_pos</topic>
-    </plugin>
-    <plugin filename="gz-sim-joint-position-controller-system" name="gz::sim::systems::JointPositionController">
       <joint_name>rudder_joint</joint_name>
       <topic>/modimoop/cmd/rudder_pos</topic>
